File: hardware/main/psu/3V3_rail.kicad_sch (KiCad schematic)
At the start: 16 parts, among them U7 LMR38025SQDRRRQ1

Commit message: expanded main pcb schematics
Parts:
- renumbered C26 to C10, C27 to C11, C28 to C12, C29 to C13, C25 to C7, C24 to C8, C23 to C9, L2 to L1, R22 to R10, R24 to R5, R19 to R6, R23 to R7, R20 to R8, R21 to R9, TP6 to TP4, U7 to U3
Changed lines of the file:
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@@
 		(in_pos_files yes)
 		(dnp no)
-		(property "Reference" "C26"
+		(property "Reference" "C10"
 			(at 156.464 83.312 0)
 			(show_name no)
@@
 			(project "main"
 				(path "/3c4b33ec-0bb0-4c39-b9f2-8186a131a3d5/b60627e7-4f8f-4feb-bf39-03b594544918/6f893b19-301a-4780-9a1e-038b0ac5ede2"
-					(reference "C26")
+					(reference "C10")
 					(unit 1)
 				)
@@
 		(in_pos_files yes)
 		(dnp no)
-		(property "Reference" "R23"
+		(property "Reference" "R7"
 			(at 121.92 107.442 90)
 			(show_name no)
@@
 			(project "main"
 				(path "/3c4b33ec-0bb0-4c39-b9f2-8186a131a3d5/b60627e7-4f8f-4feb-bf39-03b594544918/6f893b19-301a-4780-9a1e-038b0ac5ede2"
-					(reference "R23")
+					(reference "R7")
 					(unit 1)
 				)
@@
 		(in_pos_files yes)
 		(dnp no)
-		(property "Reference" "R19"
+		(property "Reference" "R6"
 			(at 120.904 99.822 0)
 			(show_name no)
@@
 			(project "main"
 				(path "/3c4b33ec-0bb0-4c39-b9f2-8186a131a3d5/b60627e7-4f8f-4feb-bf39-03b594544918/6f893b19-301a-4780-9a1e-038b0ac5ede2"
-					(reference "R19")
+					(reference "R6")
 					(unit 1)
 				)
@@
 		(in_pos_files yes)
 		(dnp no)
-		(property "Reference" "C24"
+		(property "Reference" "C8"
 			(at 97.028 98.552 0)
 			(show_name no)
@@
 			(project "main"
 				(path "/3c4b33ec-0bb0-4c39-b9f2-8186a131a3d5/b60627e7-4f8f-4feb-bf39-03b594544918/6f893b19-301a-4780-9a1e-038b0ac5ede2"
-					(reference "C24")
+					(reference "C8")
 					(unit 1)
 				)
@@
 		(in_pos_files yes)
 		(dnp no)
-		(property "Reference" "#PWR036"
+		(property "Reference" "#PWR017"
 			(at 189.23 110.49 0)
 			(hide yes)
@@
 			(project "main"
 				(path "/3c4b33ec-0bb0-4c39-b9f2-8186a131a3d5/b60627e7-4f8f-4feb-bf39-03b594544918/6f893b19-301a-4780-9a1e-038b0ac5ede2"
-					(reference "#PWR036")
+					(reference "#PWR017")
 					(unit 1)
 				)
@@
 		(in_pos_files yes)
 		(dnp no)
-		(property "Reference" "L2"
+		(property "Reference" "L1"
 			(at 162.56 92.964 90)
 			(show_name no)
@@
 			(project "main"
 				(path "/3c4b33ec-0bb0-4c39-b9f2-8186a131a3d5/b60627e7-4f8f-4feb-bf39-03b594544918/6f893b19-301a-4780-9a1e-038b0ac5ede2"
-					(reference "L2")
+					(reference "L1")
 					(unit 1)
 				)
@@
 		(in_pos_files yes)
 		(dnp no)
-		(property "Reference" "R22"
+		(property "Reference" "R10"
 			(at 169.672 108.966 0)
 			(show_name no)
@@
 			(project "main"
 				(path "/3c4b33ec-0bb0-4c39-b9f2-8186a131a3d5/b60627e7-4f8f-4feb-bf39-03b594544918/6f893b19-301a-4780-9a1e-038b0ac5ede2"
-					(reference "R22")
+					(reference "R10")
 					(unit 1)
 				)
@@
 		(in_pos_files yes)
 		(dnp no)
-		(property "Reference" "C27"
+		(property "Reference" "C11"
 			(at 179.578 101.092 0)
 			(show_name no)
@@
 			(project "main"
 				(path "/3c4b33ec-0bb0-4c39-b9f2-8186a131a3d5/b60627e7-4f8f-4feb-bf39-03b594544918/6f893b19-301a-4780-9a1e-038b0ac5ede2"
-					(reference "C27")
+					(reference "C11")
 					(unit 1)
 				)
@@
 		(in_pos_files yes)
 		(dnp no)
-		(property "Reference" "R20"
+		(property "Reference" "R8"
 			(at 156.21 98.552 90)
 			(show_name no)
@@
 			(project "main"
 				(path "/3c4b33ec-0bb0-4c39-b9f2-8186a131a3d5/b60627e7-4f8f-4feb-bf39-03b594544918/6f893b19-301a-4780-9a1e-038b0ac5ede2"
-					(reference "R20")
+					(reference "R8")
 					(unit 1)
 				)
@@
 		(dnp no)
 		(fields_autoplaced yes)
-		(property "Reference" "U7"
+		(property "Reference" "U3"
 			(at 138.43 81.28 0)
 			(show_name no)
@@
 			(project "main"
 				(path "/3c4b33ec-0bb0-4c39-b9f2-8186a131a3d5/b60627e7-4f8f-4feb-bf39-03b594544918/6f893b19-301a-4780-9a1e-038b0ac5ede2"
-					(reference "U7")
+					(reference "U3")
 					(unit 1)
 				)
@@
 		(dnp no)
 		(fields_autoplaced yes)
-		(property "Reference" "TP6"
+		(property "Reference" "TP4"
 			(at 199.39 86.8679 0)
 			(show_name no)
@@
 			(project "main"
 				(path "/3c4b33ec-0bb0-4c39-b9f2-8186a131a3d5/b60627e7-4f8f-4feb-bf39-03b594544918/6f893b19-301a-4780-9a1e-038b0ac5ede2"
-					(reference "TP6")
+					(reference "TP4")
 					(unit 1)
 				)
@@
 		(in_pos_files yes)
 		(dnp no)
-		(property "Reference" "R24"
+		(property "Reference" "R5"
 			(at 102.87 108.712 90)
 			(show_name no)
@@
 			(project "main"
 				(path "/3c4b33ec-0bb0-4c39-b9f2-8186a131a3d5/b60627e7-4f8f-4feb-bf39-03b594544918/6f893b19-301a-4780-9a1e-038b0ac5ede2"
-					(reference "R24")
+					(reference "R5")
 					(unit 1)
 				)
@@
 		(in_pos_files yes)
 		(dnp no)
-		(property "Reference" "#PWR035"
+		(property "Reference" "#PWR016"
 			(at 172.72 116.84 0)
 			(hide yes)
@@
 			(project "main"
 				(path "/3c4b33ec-0bb0-4c39-b9f2-8186a131a3d5/b60627e7-4f8f-4feb-bf39-03b594544918/6f893b19-301a-4780-9a1e-038b0ac5ede2"
-					(reference "#PWR035")
+					(reference "#PWR016")
 					(unit 1)
 				)
@@
 		(in_pos_files yes)
 		(dnp no)
-		(property "Reference" "C25"
+		(property "Reference" "C7"
 			(at 89.408 98.552 0)
 			(show_name no)
@@
 			(project "main"
 				(path "/3c4b33ec-0bb0-4c39-b9f2-8186a131a3d5/b60627e7-4f8f-4feb-bf39-03b594544918/6f893b19-301a-4780-9a1e-038b0ac5ede2"
-					(reference "C25")
+					(reference "C7")
 					(unit 1)
 				)
@@
 		(in_pos_files yes)
 		(dnp no)
-		(property "Reference" "#PWR034"
+		(property "Reference" "#PWR013"
 			(at 118.11 107.95 0)
 			(hide yes)
@@
 			(project "main"
 				(path "/3c4b33ec-0bb0-4c39-b9f2-8186a131a3d5/b60627e7-4f8f-4feb-bf39-03b594544918/6f893b19-301a-4780-9a1e-038b0ac5ede2"
-					(reference "#PWR034")
+					(reference "#PWR013")
 					(unit 1)
 				)
@@
 		(in_pos_files yes)
 		(dnp no)
-		(property "Reference" "C28"
+		(property "Reference" "C12"
 			(at 187.198 101.092 0)
 			(show_name no)
@@
 			(project "main"
 				(path "/3c4b33ec-0bb0-4c39-b9f2-8186a131a3d5/b60627e7-4f8f-4feb-bf39-03b594544918/6f893b19-301a-4780-9a1e-038b0ac5ede2"
-					(reference "C28")
+					(reference "C12")
 					(unit 1)
 				)
@@
 		(in_pos_files yes)
 		(dnp no)
-		(property "Reference" "C29"
+		(property "Reference" "C13"
 			(at 194.818 101.092 0)
 			(show_name no)
@@
 			(project "main"
 				(path "/3c4b33ec-0bb0-4c39-b9f2-8186a131a3d5/b60627e7-4f8f-4feb-bf39-03b594544918/6f893b19-301a-4780-9a1e-038b0ac5ede2"
-					(reference "C29")
+					(reference "C13")
 					(unit 1)
 				)
@@
 		(in_pos_files yes)
 		(dnp no)
-		(property "Reference" "C23"
+		(property "Reference" "C9"
 			(at 104.648 98.552 0)
 			(show_name no)
@@
 			(project "main"
 				(path "/3c4b33ec-0bb0-4c39-b9f2-8186a131a3d5/b60627e7-4f8f-4feb-bf39-03b594544918/6f893b19-301a-4780-9a1e-038b0ac5ede2"
-					(reference "C23")
+					(reference "C9")
 					(unit 1)
 				)
@@
 		(in_pos_files yes)
 		(dnp no)
-		(property "Reference" "R21"
+		(property "Reference" "R9"
 			(at 169.926 101.092 0)
 			(show_name no)
@@
 			(project "main"
 				(path "/3c4b33ec-0bb0-4c39-b9f2-8186a131a3d5/b60627e7-4f8f-4feb-bf39-03b594544918/6f893b19-301a-4780-9a1e-038b0ac5ede2"
-					(reference "R21")
+					(reference "R9")
 					(unit 1)
 				)
@@
 		(in_pos_files yes)
 		(dnp no)
-		(property "Reference" "#PWR032"
+		(property "Reference" "#PWR012"
 			(at 99.06 109.22 0)
 			(hide yes)
@@
 			(project "main"
 				(path "/3c4b33ec-0bb0-4c39-b9f2-8186a131a3d5/b60627e7-4f8f-4feb-bf39-03b594544918/6f893b19-301a-4780-9a1e-038b0ac5ede2"
-					(reference "#PWR032")
+					(reference "#PWR012")
 					(unit 1)
 				)
@@
 		(in_pos_files yes)
 		(dnp no)
-		(property "Reference" "#PWR033"
+		(property "Reference" "#PWR015"
 			(at 138.43 115.57 0)
 			(hide yes)
@@
 			(project "main"
 				(path "/3c4b33ec-0bb0-4c39-b9f2-8186a131a3d5/b60627e7-4f8f-4feb-bf39-03b594544918/6f893b19-301a-4780-9a1e-038b0ac5ede2"
-					(reference "#PWR033")
+					(reference "#PWR015")
 					(unit 1)
 				)
@@
 		(in_pos_files yes)
 		(dnp no)
-		(property "Reference" "#PWR037"
+		(property "Reference" "#PWR014"
 			(at 125.73 102.87 0)
 			(hide yes)
@@
 			(project "main"
 				(path "/3c4b33ec-0bb0-4c39-b9f2-8186a131a3d5/b60627e7-4f8f-4feb-bf39-03b594544918/6f893b19-301a-4780-9a1e-038b0ac5ede2"
-					(reference "#PWR037")
-					(unit 1)
-				)
+					(reference "#PWR014")
+					(unit 1)
+				)
