File: hardware/main/psu/5V_rail.kicad_sch (KiCad schematic)
At the start: 24 parts, among them U6 LM70840QRRXRQ1

Commit message: expanded main pcb schematics
Parts:
- renumbered C18 to C14, C17 to C15, C21 to C16, C22 to C17, C12 to C18, C15 to C19, C14 to C20, C11 to C21, C16 to C22, C20 to C23, C19 to C24, L1 to L2, R25 to R11, R18 to R12, R17 to R13, R10 to R14, R13 to R15, R14 to R16, R11 to R17, R9 to R18, R12 to R19, R15 to R20, U6 to U4

Commit message: fixed ERC issues
Parts:
- added NT1: NetTie_2, symbol Device:NetTie_2
Connections:
- net GND: now also NT1.2; no longer C19.1, C20.2, C22.1, U4.17 (AGND), U4.8 (PFM/SYNCIN)
- new net GNDA: C19.1, C20.2, C22.1, NT1.1, U4.17 (AGND), U4.8 (PFM/SYNCIN)
- no-connect marks 0 -> 1
