File: hardware/main/psu/PSU_controller.kicad_sch (KiCad schematic)
At the start: 30 parts, among them J2 Conn_01x03_Pin, Q2 2N7002, Q3 2N7002, Q4 2N7002, Q5 2N7002, U2 ATtiny1616-M, U4 74LVC1G74, U5 TLV803E

Commit message: expanded main pcb schematics
Parts:
- renumbered C9 to C26, C7 to C27, C8 to C28, C10 to C29, D4 to D6, D3 to D7, Q4 to Q2, Q5 to Q3, Q3 to Q4, Q2 to Q5, R4 to R22, R3 to R23, R28 to R24, R31 to R25, R5 to R26, R26 to R27, R29 to R28, R30 to R29, R8 to R30, R7 to R31, R6 to R32, R16 to R33, TP9 to TP10, TP10 to TP9, U2 to U6, U5 to U7, U4 to U8

Commit message: fixed ERC issues
Connections:
- no-connect marks 1 -> 13
Changed lines of the file:
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@@
+	)
+	(no_connect
+		(at 137.16 87.63)
+	)
+	(no_connect
+		(at 137.16 85.09)
+	)
+	(no_connect
+		(at 137.16 97.79)
 	)
 	(no_connect
 		(at 196.85 107.95)
+	)
+	(no_connect
+		(at 137.16 105.41)
+	)
+	(no_connect
+		(at 137.16 100.33)
+	)
+	(no_connect
+		(at 137.16 77.47)
+	)
+	(no_connect
+		(at 137.16 102.87)
+	)
+	(no_connect
+		(at 106.68 100.33)
+	)
+	(no_connect
+		(at 137.16 82.55)
+	)
+	(no_connect
+		(at 137.16 72.39)
+	)
+	(no_connect
+		(at 137.16 80.01)
+	)
+	(no_connect
+		(at 137.16 74.93)
 	)
 	(wire
@@
 		)
 	)
-	(label "To Pi GPIO with 10k pull-up to pi 3V3"
-		(at 59.69 157.48 0)
-		(effects
-			(font
-				(size 1.27 1.27)
-			)
-			(justify left bottom)
-		)
-	)
 	(label "PSU_ON"
 		(at 149.86 118.11 0)
 		(effects
 			(font
-				(size 1.27 1.27)
-			)
-			(justify left bottom)
-		)
-	)
-	(label "Set LOW to power off"
-		(at 139.7 128.27 0)
-		(effects
-			(font
