File: hardware/main/psu/power_supply.kicad_sch (KiCad schematic)
At the start: 13 parts, among them J1 Power 3-Pin, U8 TMP112xxDRL

Commit message: expanded main pcb schematics
Parts:
- renumbered C13 to C1, D2 to D1, D5 to D2, D6 to D3, D7 to D4, R33 to R1, R27 to R2, R32 to R3, TP3 to TP1, TP4 to TP2, U8 to U1
Changed lines of the file:
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@@
+	(wire
+		(pts
+			(xy 111.76 111.76) (xy 124.46 111.76)
+		)
+		(stroke
+			(width 0)
+			(type default)
+		)
+	)
 	(wire
 		(pts
@@
 		(pts
 			(xy 184.15 139.7) (xy 185.42 139.7)
+		)
+		(stroke
+			(width 0)
+			(type default)
+		)
+	)
+	(wire
+		(pts
+			(xy 111.76 106.68) (xy 124.46 106.68)
 		)
 		(stroke
@@
 		)
 	)
+	(hierarchical_label "PI_OFF_SIGNAL"
+		(shape input)
+		(at 111.76 111.76 180)
+		(effects
+			(font
+				(size 1.27 1.27)
+			)
+			(justify right)
+		)
+	)
 	(hierarchical_label "SDA"
 		(shape bidirectional)
@@
 			)
 			(justify left)
+		)
+	)
+	(hierarchical_label "PI_OFF_REQUEST"
+		(shape output)
+		(at 111.76 106.68 180)
+		(effects
+			(font
+				(size 1.27 1.27)
+			)
+			(justify right)
 		)
 	)
@@
 		(dnp no)
 		(fields_autoplaced yes)
-		(property "Reference" "U8"
+		(property "Reference" "U1"
 			(at 220.98 109.1498 0)
 			(show_name no)
@@
 			(project "main"
 				(path "/3c4b33ec-0bb0-4c39-b9f2-8186a131a3d5/b60627e7-4f8f-4feb-bf39-03b594544918"
-					(reference "U8")
+					(reference "U1")
 					(unit 1)
 				)
@@
 		(in_pos_files yes)
 		(dnp no)
-		(property "Reference" "#PWR041"
+		(property "Reference" "#PWR06"
 			(at 208.28 86.36 0)
 			(hide yes)
@@
 			(project "main"
 				(path "/3c4b33ec-0bb0-4c39-b9f2-8186a131a3d5/b60627e7-4f8f-4feb-bf39-03b594544918"
-					(reference "#PWR041")
+					(reference "#PWR06")
 					(unit 1)
 				)
@@
 		(in_pos_files yes)
 		(dnp no)
-		(property "Reference" "#PWR043"
+		(property "Reference" "#PWR03"
 			(at 189.23 113.03 0)
 			(hide yes)
@@
 			(project "main"
 				(path "/3c4b33ec-0bb0-4c39-b9f2-8186a131a3d5/b60627e7-4f8f-4feb-bf39-03b594544918"
-					(reference "#PWR043")
+					(reference "#PWR03")
 					(unit 1)
 				)
@@
 		(in_pos_files yes)
 		(dnp no)
-		(property "Reference" "#PWR042"
+		(property "Reference" "#PWR05"
 			(at 205.74 137.16 0)
 			(hide yes)
@@
 			(project "main"
 				(path "/3c4b33ec-0bb0-4c39-b9f2-8186a131a3d5/b60627e7-4f8f-4feb-bf39-03b594544918"
-					(reference "#PWR042")
+					(reference "#PWR05")
 					(unit 1)
 				)
@@
 		(dnp no)
 		(fields_autoplaced yes)
-		(property "Reference" "R27"
+		(property "Reference" "R2"
 			(at 232.41 138.4299 0)
 			(show_name no)
@@
 			(project "main"
 				(path "/3c4b33ec-0bb0-4c39-b9f2-8186a131a3d5/b60627e7-4f8f-4feb-bf39-03b594544918"
-					(reference "R27")
+					(reference "R2")
 					(unit 1)
 				)
@@
 		(dnp no)
 		(fields_autoplaced yes)
-		(property "Reference" "#PWR04"
+		(property "Reference" "#PWR01"
 			(at 57.15 82.55 0)
 			(hide yes)
@@
 			(project "main"
 				(path "/3c4b33ec-0bb0-4c39-b9f2-8186a131a3d5/b60627e7-4f8f-4feb-bf39-03b594544918"
-					(reference "#PWR04")
+					(reference "#PWR01")
 					(unit 1)
 				)
@@
 		(in_pos_files yes)
 		(dnp no)
-		(property "Reference" "#PWR044"
+		(property "Reference" "#PWR04"
 			(at 191.77 129.54 0)
 			(hide yes)
@@
 			(project "main"
 				(path "/3c4b33ec-0bb0-4c39-b9f2-8186a131a3d5/b60627e7-4f8f-4feb-bf39-03b594544918"
-					(reference "#PWR044")
+					(reference "#PWR04")
 					(unit 1)
 				)
@@
 		(in_pos_files yes)
 		(dnp no)
-		(property "Reference" "TP3"
+		(property "Reference" "TP1"
 			(at 50.038 84.582 0)
 			(show_name no)
@@
 			(project "main"
 				(path "/3c4b33ec-0bb0-4c39-b9f2-8186a131a3d5/b60627e7-4f8f-4feb-bf39-03b594544918"
-					(reference "TP3")
+					(reference "TP1")
 					(unit 1)
 				)
@@
 		(in_pos_files yes)
 		(dnp no)
-		(property "Reference" "C13"
+		(property "Reference" "C1"
 			(at 202.946 109.728 90)
 			(show_name no)
@@
 			(project "main"
 				(path "/3c4b33ec-0bb0-4c39-b9f2-8186a131a3d5/b60627e7-4f8f-4feb-bf39-03b594544918"
-					(reference "C13")
+					(reference "C1")
 					(unit 1)
 				)
@@
 		(in_pos_files yes)
 		(dnp no)
-		(property "Reference" "#PWR07"
+		(property "Reference" "#PWR02"
 			(at 71.12 99.06 0)
 			(hide yes)
@@
 			(project "main"
 				(path "/3c4b33ec-0bb0-4c39-b9f2-8186a131a3d5/b60627e7-4f8f-4feb-bf39-03b594544918"
-					(reference "#PWR07")
+					(reference "#PWR02")
 					(unit 1)
 				)
@@
 		(in_pos_files yes)
 		(dnp no)
-		(property "Reference" "D5"
+		(property "Reference" "D2"
 			(at 175.5775 57.15 0)
 			(show_name no)
@@
 			(project "main"
 				(path "/3c4b33ec-0bb0-4c39-b9f2-8186a131a3d5/b60627e7-4f8f-4feb-bf39-03b594544918"
-					(reference "D5")
+					(reference "D2")
 					(unit 1)
 				)
@@
 		(dnp no)
 		(fields_autoplaced yes)
-		(property "Reference" "D6"
+		(property "Reference" "D3"
 			(at 232.41 130.4924 90)
 			(show_name no)
@@
 			(project "main"
 				(path "/3c4b33ec-0bb0-4c39-b9f2-8186a131a3d5/b60627e7-4f8f-4feb-bf39-03b594544918"
-					(reference "D6")
+					(reference "D3")
 					(unit 1)
 				)
@@
 		(dnp no)
 		(fields_autoplaced yes)
-		(property "Reference" "D2"
+		(property "Reference" "D1"
 			(at 73.66 87.6299 90)
 			(show_name no)
@@
 			(project "main"
 				(path "/3c4b33ec-0bb0-4c39-b9f2-8186a131a3d5/b60627e7-4f8f-4feb-bf39-03b594544918"
-					(reference "D2")
+					(reference "D1")
 					(unit 1)
 				)
@@
 		(dnp no)
 		(fields_autoplaced yes)
-		(property "Reference" "R33"
+		(property "Reference" "R1"
 			(at 163.83 58.42 90)
 			(show_name no)
@@
 			(project "main"
 				(path "/3c4b33ec-0bb0-4c39-b9f2-8186a131a3d5/b60627e7-4f8f-4feb-bf39-03b594544918"
-					(reference "R33")
+					(reference "R1")
 					(unit 1)
 				)
@@
 		(in_pos_files yes)
 		(dnp no)
-		(property "Reference" "TP4"
+		(property "Reference" "TP2"
 			(at 56.388 58.928 0)
 			(show_name no)
@@
 			(project "main"
 				(path "/3c4b33ec-0bb0-4c39-b9f2-8186a131a3d5/b60627e7-4f8f-4feb-bf39-03b594544918"
-					(reference "TP4")
+					(reference "TP2")
 					(unit 1)
 				)
@@
 		(dnp no)
 		(fields_autoplaced yes)
-		(property "Reference" "D7"
+		(property "Reference" "D4"
 			(at 234.95 83.5024 90)
 			(show_name no)
@@
 			(project "main"
 				(path "/3c4b33ec-0bb0-4c39-b9f2-8186a131a3d5/b60627e7-4f8f-4feb-bf39-03b594544918"
-					(reference "D7")
+					(reference "D4")
 					(unit 1)
 				)
@@
 		(dnp no)
 		(fields_autoplaced yes)
-		(property "Reference" "R32"
+		(property "Reference" "R3"
 			(at 234.95 91.4399 0)
 			(show_name no)
@@
 			(project "main"
 				(path "/3c4b33ec-0bb0-4c39-b9f2-8186a131a3d5/b60627e7-4f8f-4feb-bf39-03b594544918"
-					(reference "R32")
+					(reference "R3")
 					(unit 1)
 				)
@@
 		(in_pos_files yes)
 		(dnp no)
-		(property "Reference" "#PWR045"
+		(property "Reference" "#PWR07"
 			(at 218.44 121.92 0)
 			(hide yes)
@@
 			(project "main"
 				(path "/3c4b33ec-0bb0-4c39-b9f2-8186a131a3d5/b60627e7-4f8f-4feb-bf39-03b594544918"
-					(reference "#PWR045")
+					(reference "#PWR07")
 					(unit 1)
 				)

Commit message: fixed ERC issues
Connections:
- net GND: no longer U1.3 (ALERT)
- no-connect marks 0 -> 1
Other:
- note added: "BTN"
- note added: "GND"
- note added: "IGN"
