File: hardware/main/psu/protection_circuit.kicad_sch (KiCad schematic)
At the start: 11 parts, among them Q1 DMT6007LFG-13, U1 LM74700

Commit message: expanded main pcb schematics
Parts:
- renumbered C1 to C2, C5 to C3, C2 to C5, C3 to C6, D1 to D5, R1 to R4, TP1 to TP3, U1 to U2
Changed lines of the file:
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@@
 		(in_pos_files yes)
 		(dnp no)
-		(property "Reference" "C1"
+		(property "Reference" "C2"
 			(at 135.89 93.726 90)
 			(show_name no)
@@
 			(project "main"
 				(path "/3c4b33ec-0bb0-4c39-b9f2-8186a131a3d5/b60627e7-4f8f-4feb-bf39-03b594544918/506fecb8-81d5-49f3-ae59-2c4b2d066e9f"
-					(reference "C1")
+					(reference "C2")
 					(unit 1)
 				)
@@
 		(dnp no)
 		(fields_autoplaced yes)
-		(property "Reference" "U1"
+		(property "Reference" "U2"
 			(at 163.83 97.7899 0)
 			(show_name no)
@@
 			(project "main"
 				(path "/3c4b33ec-0bb0-4c39-b9f2-8186a131a3d5/b60627e7-4f8f-4feb-bf39-03b594544918/506fecb8-81d5-49f3-ae59-2c4b2d066e9f"
-					(reference "U1")
+					(reference "U2")
 					(unit 1)
 				)
@@
 		(in_pos_files yes)
 		(dnp no)
-		(property "Reference" "R1"
+		(property "Reference" "R4"
 			(at 136.144 108.204 90)
 			(show_name no)
@@
 			(project "main"
 				(path "/3c4b33ec-0bb0-4c39-b9f2-8186a131a3d5/b60627e7-4f8f-4feb-bf39-03b594544918/506fecb8-81d5-49f3-ae59-2c4b2d066e9f"
-					(reference "R1")
+					(reference "R4")
 					(unit 1)
 				)
@@
 		(dnp no)
 		(fields_autoplaced yes)
-		(property "Reference" "#PWR06"
+		(property "Reference" "#PWR09"
 			(at 143.51 71.12 0)
 			(hide yes)
@@
 			(project "main"
 				(path "/3c4b33ec-0bb0-4c39-b9f2-8186a131a3d5/b60627e7-4f8f-4feb-bf39-03b594544918/506fecb8-81d5-49f3-ae59-2c4b2d066e9f"
-					(reference "#PWR06")
+					(reference "#PWR09")
 					(unit 1)
 				)
@@
 		(in_pos_files yes)
 		(dnp no)
-		(property "Reference" "C3"
+		(property "Reference" "C6"
 			(at 192.278 74.168 0)
 			(show_name no)
@@
 			(project "main"
 				(path "/3c4b33ec-0bb0-4c39-b9f2-8186a131a3d5/b60627e7-4f8f-4feb-bf39-03b594544918/506fecb8-81d5-49f3-ae59-2c4b2d066e9f"
-					(reference "C3")
+					(reference "C6")
 					(unit 1)
 				)
@@
 		(in_pos_files yes)
 		(dnp no)
-		(property "Reference" "#PWR05"
+		(property "Reference" "#PWR011"
 			(at 182.88 60.96 0)
 			(hide yes)
@@
 			(project "main"
 				(path "/3c4b33ec-0bb0-4c39-b9f2-8186a131a3d5/b60627e7-4f8f-4feb-bf39-03b594544918/506fecb8-81d5-49f3-ae59-2c4b2d066e9f"
-					(reference "#PWR05")
+					(reference "#PWR011")
 					(unit 1)
 				)
@@
 		(dnp no)
 		(fields_autoplaced yes)
-		(property "Reference" "D1"
+		(property "Reference" "D5"
 			(at 116.84 95.2499 90)
 			(show_name no)
@@
 			(project "main"
 				(path "/3c4b33ec-0bb0-4c39-b9f2-8186a131a3d5/b60627e7-4f8f-4feb-bf39-03b594544918/506fecb8-81d5-49f3-ae59-2c4b2d066e9f"
-					(reference "D1")
+					(reference "D5")
 					(unit 1)
 				)
@@
 		(dnp no)
 		(fields_autoplaced yes)
-		(property "Reference" "TP1"
+		(property "Reference" "TP3"
 			(at 209.55 70.3579 0)
 			(show_name no)
@@
 			(project "main"
 				(path "/3c4b33ec-0bb0-4c39-b9f2-8186a131a3d5/b60627e7-4f8f-4feb-bf39-03b594544918/506fecb8-81d5-49f3-ae59-2c4b2d066e9f"
-					(reference "TP1")
+					(reference "TP3")
 					(unit 1)
 				)
@@
 		(dnp no)
 		(fields_autoplaced yes)
-		(property "Reference" "#PWR02"
+		(property "Reference" "#PWR08"
 			(at 114.3 107.95 0)
 			(hide yes)
@@
 			(project "main"
 				(path "/3c4b33ec-0bb0-4c39-b9f2-8186a131a3d5/b60627e7-4f8f-4feb-bf39-03b594544918/506fecb8-81d5-49f3-ae59-2c4b2d066e9f"
-					(reference "#PWR02")
+					(reference "#PWR08")
 					(unit 1)
 				)
@@
 		(in_pos_files yes)
 		(dnp no)
-		(property "Reference" "C2"
+		(property "Reference" "C5"
 			(at 183.642 74.168 0)
 			(show_name no)
@@
 			(project "main"
 				(path "/3c4b33ec-0bb0-4c39-b9f2-8186a131a3d5/b60627e7-4f8f-4feb-bf39-03b594544918/506fecb8-81d5-49f3-ae59-2c4b2d066e9f"
-					(reference "C2")
+					(reference "C5")
 					(unit 1)
 				)
@@
 		(dnp no)
 		(fields_autoplaced yes)
-		(property "Reference" "#PWR03"
+		(property "Reference" "#PWR010"
 			(at 152.4 115.57 0)
 			(hide yes)
@@
 			(project "main"
 				(path "/3c4b33ec-0bb0-4c39-b9f2-8186a131a3d5/b60627e7-4f8f-4feb-bf39-03b594544918/506fecb8-81d5-49f3-ae59-2c4b2d066e9f"
-					(reference "#PWR03")
+					(reference "#PWR010")
 					(unit 1)
 				)
@@
 		(in_pos_files yes)
 		(dnp no)
-		(property "Reference" "C5"
+		(property "Reference" "C3"
 			(at 144.272 86.614 0)
 			(show_name no)
@@
 			(project "main"
 				(path "/3c4b33ec-0bb0-4c39-b9f2-8186a131a3d5/b60627e7-4f8f-4feb-bf39-03b594544918/506fecb8-81d5-49f3-ae59-2c4b2d066e9f"
-					(reference "C5")
-					(unit 1)
-				)
+					(reference "C3")
+					(unit 1)
+				)

Commit message: fixed ERC issues
Changed lines of the file:
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@@
-		)
-	)
-	(label "Caps with 100V ratings"
-		(at 113.03 83.82 0)
-		(effects
-			(font
-				(size 1.27 1.27)
-			)
-			(justify left bottom)
 		)
 	)
