File: hardware/main/sensors/sensors.kicad_sch (KiCad schematic)
At the start: 21 parts, among them J1 Conn_01x02, J2 Conn_01x02, U1 ADS1115IDGS

Commit message: expanded main pcb schematics
Parts:
- renumbered C2 to C42, C3 to C43, C4 to C44, C1 to C45, C5 to C46, D7 to D10, D8 to D11, D5 to D12, D6 to D13, D4 to D8, D3 to D9, J2 to J4, J1 to J5, R2 to R45, R4 to R46, R1 to R47, R3 to R48, R5 to R49, R7 to R50, R6 to R51, U1 to U13
