File: hardware/main/can.kicad_sch (KiCad schematic)
At the start: 11 parts, among them J3 Conn_02x02_Odd_Even, U11 MCP2515-xST, U12 PTCAN3404DDFRQ1, Y1 16MHz

Commit message: fixed ERC issues
Parts:
- removed U12: PTCAN3404DDFRQ1, DDF0008A-IPC_A, symbol TCAN3404-Q1:PTCAN3404DDFRQ1
- added U16: PTCAN3404DDFRQ1, TCAN3404-Q1:DDF0008A-IPC_A, symbol TCAN3404-Q1:PTCAN3404DDFRQ1
- CR1: footprint SOT-23_DBZ_TEX -> ESD2CAN24-Q1:SOT-23_DBZ_TEX
Connections:
- net 3V3_RAIL: now also U16.3 (VCC)
- net GND: now also U16.2 (GND), U16.5 (SHDN), U16.8 (STB)
- net at CR1.1, J3.1 (Pin_1): now also U16.7 (CANH)
- net at CR1.2, J3.3 (Pin_3): now also U16.6 (CANL)
- net at U11.1 (TXCAN): now also U16.1 (TXD)
- net at U11.2 (RXCAN): now also U16.4 (RXD)
Changed lines of the file:
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@@
-	)
-	(symbol
-		(lib_id "TCAN3404-Q1:PTCAN3404DDFRQ1")
-		(at 151.13 87.63 0)
-		(unit 1)
-		(body_style 1)
-		(exclude_from_sim no)
-		(in_bom yes)
-		(on_board yes)
-		(in_pos_files yes)
-		(dnp no)
-		(fields_autoplaced yes)
-		(property "Reference" "U12"
-			(at 168.91 77.47 0)
-			(show_name no)
-			(do_not_autoplace no)
-			(effects
-				(font
-					(size 1.524 1.524)
-				)
-			)
-		)
-		(property "Value" "PTCAN3404DDFRQ1"
-			(at 168.91 80.01 0)
-			(show_name no)
-			(do_not_autoplace no)
-			(effects
-				(font
-					(size 1.524 1.524)
-				)
-			)
-		)
-		(property "Footprint" "DDF0008A-IPC_A"
-			(at 151.13 87.63 0)
-			(hide yes)
-			(show_name no)
-			(do_not_autoplace no)
-			(effects
-				(font
-					(size 1.27 1.27)
-					(italic yes)
-				)
-			)
-		)
-		(property "Datasheet" "https://www.ti.com/lit/gpn/tcan3404-q1"
-			(at 151.13 87.63 0)
-			(hide yes)
-			(show_name no)
-			(do_not_autoplace no)
-			(effects
-				(font
-					(size 1.27 1.27)
-					(italic yes)
-				)
-			)
-		)
-		(property "Description" ""
-			(at 151.13 87.63 0)
-			(hide yes)
-			(show_name no)
-			(do_not_autoplace no)
-			(effects
-				(font
-					(size 1.27 1.27)
-				)
-			)
-		)
-		(pin "5"
-		)
-		(pin "7"
-		)
-		(pin "1"
-		)
-		(pin "2"
-		)
-		(pin "3"
-		)
-		(pin "4"
-		)
-		(pin "6"
-		)
-		(pin "8"
-		)
-		(instances
-			(project "main"
-				(path "/3c4b33ec-0bb0-4c39-b9f2-8186a131a3d5/9ae84d67-064b-4531-bc2c-ef16eda37330"
-					(reference "U12")
-					(unit 1)
-				)
-			)
-		)
 	)
 	(symbol
@@
 	)
 	(symbol
+		(lib_id "TCAN3404-Q1:PTCAN3404DDFRQ1")
+		(at 151.13 87.63 0)
+		(unit 1)
+		(body_style 1)
+		(exclude_from_sim no)
+		(in_bom yes)
+		(on_board yes)
+		(in_pos_files yes)
+		(dnp no)
+		(fields_autoplaced yes)
+		(property "Reference" "U16"
+			(at 168.91 77.47 0)
+			(show_name no)
+			(do_not_autoplace no)
+			(effects
+				(font
+					(size 1.524 1.524)
+				)
+			)
+		)
+		(property "Value" "PTCAN3404DDFRQ1"
+			(at 168.91 80.01 0)
+			(show_name no)
+			(do_not_autoplace no)
+			(effects
+				(font
+					(size 1.524 1.524)
+				)
+			)
+		)
+		(property "Footprint" "TCAN3404-Q1:DDF0008A-IPC_A"
+			(at 151.13 87.63 0)
+			(hide yes)
+			(show_name no)
+			(do_not_autoplace no)
+			(effects
+				(font
+					(size 1.27 1.27)
+					(italic yes)
+				)
+			)
+		)
+		(property "Datasheet" "https://www.ti.com/lit/gpn/tcan3404-q1"
+			(at 151.13 87.63 0)
+			(hide yes)
+			(show_name no)
+			(do_not_autoplace no)
+			(effects
+				(font
+					(size 1.27 1.27)
+					(italic yes)
+				)
+			)
+		)
+		(property "Description" ""
+			(at 151.13 87.63 0)
+			(hide yes)
+			(show_name no)
+			(do_not_autoplace no)
+			(effects
+				(font
+					(size 1.27 1.27)
+				)
+			)
+		)
+		(pin "6"
+		)
+		(pin "2"
+		)
+		(pin "8"
+		)
+		(pin "5"
+		)
+		(pin "1"
+		)
+		(pin "4"
+		)
+		(pin "7"
+		)
+		(pin "3"
+		)
+		(instances
+			(project "main"
+				(path "/3c4b33ec-0bb0-4c39-b9f2-8186a131a3d5/9ae84d67-064b-4531-bc2c-ef16eda37330"
+					(reference "U16")
+					(unit 1)
+				)
+			)
+		)
+	)
+	(symbol
 		(lib_id "ESD2CAN24-Q1:PESD2CAN24DBZRQ1")
 		(at 199.39 95.25 0)
@@
 			)
 		)
-		(property "Footprint" "SOT-23_DBZ_TEX"
+		(property "Footprint" "ESD2CAN24-Q1:SOT-23_DBZ_TEX"
 			(at 199.39 95.25 0)
 			(hide yes)
