File: hardware/xr25/3V3_power_supply.kicad_sch (KiCad schematic)
At the start: 14 parts, among them U2 LMR36015AQRNXRQ1

Commit message: fixed more ERC issues
Parts:
- U2: footprint RNX0012B -> LMR36015AQRNXRQ1:RNX0012B
Changed lines of the file:
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@@
+	)
+	(junction
+		(at 227.33 83.82)
+		(diameter 0)
+		(color 0 0 0 0)
 	)
 	(junction
@@
 	)
 	(junction
+		(at 97.79 76.2)
+		(diameter 0)
+		(color 0 0 0 0)
+	)
+	(junction
+		(at 86.36 76.2)
+		(diameter 0)
+		(color 0 0 0 0)
+	)
+	(junction
+		(at 118.11 100.33)
+		(diameter 0)
+		(color 0 0 0 0)
+	)
+	(junction
+		(at 212.09 104.14)
+		(diameter 0)
+		(color 0 0 0 0)
+	)
+	(junction
+		(at 97.79 91.44)
+		(diameter 0)
+		(color 0 0 0 0)
+	)
+	(junction
+		(at 223.52 83.82)
+		(diameter 0)
+		(color 0 0 0 0)
+	)
+	(junction
+		(at 212.09 83.82)
+		(diameter 0)
+		(color 0 0 0 0)
+	)
+	(junction
+		(at 182.88 83.82)
+		(diameter 0)
+		(color 0 0 0 0)
+	)
+	(junction
+		(at 118.11 91.44)
+		(diameter 0)
+		(color 0 0 0 0)
+	)
+	(junction
+		(at 190.5 83.82)
+		(diameter 0)
+		(color 0 0 0 0)
+	)
+	(junction
+		(at 109.22 91.44)
+		(diameter 0)
+		(color 0 0 0 0)
+	)
+	(junction
+		(at 200.66 83.82)
+		(diameter 0)
+		(color 0 0 0 0)
+	)
+	(junction
+		(at 109.22 76.2)
+		(diameter 0)
+		(color 0 0 0 0)
+	)
+	(junction
 		(at 168.91 83.82)
-		(diameter 0)
-		(color 0 0 0 0)
-	)
-	(junction
-		(at 97.79 76.2)
-		(diameter 0)
-		(color 0 0 0 0)
-	)
-	(junction
-		(at 86.36 76.2)
-		(diameter 0)
-		(color 0 0 0 0)
-	)
-	(junction
-		(at 118.11 100.33)
-		(diameter 0)
-		(color 0 0 0 0)
-	)
-	(junction
-		(at 212.09 104.14)
-		(diameter 0)
-		(color 0 0 0 0)
-	)
-	(junction
-		(at 97.79 91.44)
-		(diameter 0)
-		(color 0 0 0 0)
-	)
-	(junction
-		(at 223.52 83.82)
-		(diameter 0)
-		(color 0 0 0 0)
-	)
-	(junction
-		(at 212.09 83.82)
-		(diameter 0)
-		(color 0 0 0 0)
-	)
-	(junction
-		(at 182.88 83.82)
-		(diameter 0)
-		(color 0 0 0 0)
-	)
-	(junction
-		(at 118.11 91.44)
-		(diameter 0)
-		(color 0 0 0 0)
-	)
-	(junction
-		(at 190.5 83.82)
-		(diameter 0)
-		(color 0 0 0 0)
-	)
-	(junction
-		(at 109.22 91.44)
-		(diameter 0)
-		(color 0 0 0 0)
-	)
-	(junction
-		(at 200.66 83.82)
-		(diameter 0)
-		(color 0 0 0 0)
-	)
-	(junction
-		(at 109.22 76.2)
 		(diameter 0)
 		(color 0 0 0 0)
@@
 	(wire
 		(pts
+			(xy 223.52 83.82) (xy 227.33 83.82)
+		)
+		(stroke
+			(width 0)
+			(type default)
+		)
+	)
+	(wire
+		(pts
+			(xy 227.33 83.82) (xy 229.87 83.82)
+		)
+		(stroke
+			(width 0)
+			(type default)
+		)
+	)
+	(wire
+		(pts
 			(xy 223.52 86.36) (xy 223.52 83.82)
-		)
-		(stroke
-			(width 0)
-			(type default)
-		)
-	)
-	(wire
-		(pts
-			(xy 223.52 83.82) (xy 229.87 83.82)
 		)
 		(stroke
@@
 	)
 	(symbol
+		(lib_id "LMR36015AQRNXRQ1:LMR36015AQRNXRQ1")
+		(at 148.59 91.44 0)
+		(unit 1)
+		(body_style 1)
+		(exclude_from_sim no)
+		(in_bom yes)
+		(on_board yes)
+		(in_pos_files yes)
+		(dnp no)
+		(fields_autoplaced yes)
+		(property "Reference" "U2"
+			(at 148.59 66.04 0)
+			(show_name no)
+			(do_not_autoplace no)
+			(effects
+				(font
+					(size 1.524 1.524)
+				)
+			)
+		)
+		(property "Value" "LMR36015AQRNXRQ1"
+			(at 148.59 68.58 0)
+			(show_name no)
+			(do_not_autoplace no)
+			(effects
+				(font
+					(size 1.524 1.524)
+				)
+			)
+		)
+		(property "Footprint" "LMR36015AQRNXRQ1:RNX0012B"
+			(at 148.59 91.44 0)
+			(hide yes)
+			(show_name no)
+			(do_not_autoplace no)
+			(effects
+				(font
+					(size 1.27 1.27)
+					(italic yes)
+				)
+			)
+		)
+		(property "Datasheet" "https://www.ti.com/lit/gpn/lmr36015-q1"
+			(at 148.59 91.44 0)
+			(hide yes)
+			(show_name no)
+			(do_not_autoplace no)
+			(effects
+				(font
+					(size 1.27 1.27)
+					(italic yes)
+				)
+			)
+		)
+		(property "Description" ""
+			(at 148.59 91.44 0)
+			(hide yes)
+			(show_name no)
+			(do_not_autoplace no)
+			(effects
+				(font
+					(size 1.27 1.27)
+				)
+			)
+		)
+		(pin "5"
+		)
+		(pin "9"
+		)
+		(pin "2"
+		)
+		(pin "10"
+		)
+		(pin "4"
+		)
+		(pin "7"
+		)
+		(pin "12"
+		)
+		(pin "3"
+		)
+		(pin "1"
+		)
+		(pin "11"
+		)
+		(pin "8"
+		)
+		(pin "6"
+		)
+		(instances
+			(project "xr25"
+				(path "/857fcb83-ed52-4e01-bdd2-c0a4a3a1ca9a/646e837e-3db1-4305-b6ca-1f0b46325de9"
+					(reference "U2")
+					(unit 1)
+				)
+			)
+		)
+	)
+	(symbol
 		(lib_id "Device:C_Small")
 		(at 172.72 73.66 0)
@@
 	)
 	(symbol
+		(lib_id "power:PWR_FLAG")
+		(at 227.33 83.82 0)
+		(unit 1)
+		(body_style 1)
+		(exclude_from_sim no)
+		(in_bom yes)
+		(on_board yes)
+		(in_pos_files yes)
+		(dnp no)
+		(fields_autoplaced yes)
+		(property "Reference" "#FLG03"
+			(at 227.33 81.915 0)
+			(hide yes)
+			(show_name no)
+			(do_not_autoplace no)
+			(effects
+				(font
+					(size 1.27 1.27)
+				)
+			)
+		)
+		(property "Value" "PWR_FLAG"
+			(at 227.33 78.74 0)
+			(hide yes)
+			(show_name no)
+			(do_not_autoplace no)
+			(effects
+				(font
+					(size 1.27 1.27)
+				)
+			)
+		)
+		(property "Footprint" ""
+			(at 227.33 83.82 0)
+			(hide yes)
+			(show_name no)
+			(do_not_autoplace no)
+			(effects
+				(font
+					(size 1.27 1.27)
+				)
+			)
+		)
+		(property "Datasheet" ""
+			(at 227.33 83.82 0)
+			(hide yes)
+			(show_name no)
+			(do_not_autoplace no)
+			(effects
+				(font
+					(size 1.27 1.27)
+				)
+			)
+		)
+		(property "Description" "Special symbol for telling ERC where power comes from"
+			(at 227.33 83.82 0)
+			(hide yes)
+			(show_name no)
+			(do_not_autoplace no)
+			(effects
+				(font
+					(size 1.27 1.27)
+				)
+			)
+		)
+		(pin "1"
+		)
+		(instances
+			(project "xr25"
+				(path "/857fcb83-ed52-4e01-bdd2-c0a4a3a1ca9a/646e837e-3db1-4305-b6ca-1f0b46325de9"
+					(reference "#FLG03")
+					(unit 1)
+				)
+			)
+		)
+	)
+	(symbol
 		(lib_id "Device:R_Small")
 		(at 223.52 76.2 0)
@@
 					(unit 1)
 				)
-			)
-		)
-	)
-	(symbol
-		(lib_id "LMR36015AQRNXRQ1:LMR36015AQRNXRQ1")
-		(at 148.59 91.44 0)
-		(unit 1)
-		(body_style 1)
-		(exclude_from_sim no)
-		(in_bom yes)
-		(on_board yes)
-		(in_pos_files yes)
-		(dnp no)
-		(fields_autoplaced yes)
-		(property "Reference" "U2"
-			(at 148.59 66.04 0)
-			(show_name no)
-			(do_not_autoplace no)
-			(effects
-				(font
-					(size 1.524 1.524)
-				)
-			)
-		)
-		(property "Value" "LMR36015AQRNXRQ1"
-			(at 148.59 68.58 0)
-			(show_name no)
-			(do_not_autoplace no)
-			(effects
-				(font
-					(size 1.524 1.524)
-				)
-			)
-		)
-		(property "Footprint" "RNX0012B"
-			(at 148.59 91.44 0)
-			(hide yes)
-			(show_name no)
-			(do_not_autoplace no)
-			(effects
-				(font
-					(size 1.27 1.27)
-					(italic yes)
-				)
-			)
-		)
-		(property "Datasheet" "https://www.ti.com/lit/gpn/lmr36015-q1"
-			(at 148.59 91.44 0)
-			(hide yes)
-			(show_name no)
-			(do_not_autoplace no)
-			(effects
-				(font
-					(size 1.27 1.27)
-					(italic yes)
-				)
-			)
-		)
-		(property "Description" ""
-			(at 148.59 91.44 0)
-			(hide yes)
-			(show_name no)
-			(do_not_autoplace no)
-			(effects
-				(font
-					(size 1.27 1.27)
-				)
-			)
-		)
-		(pin "1"
-		)
-		(pin "2"
-		)
-		(pin "3"
-		)
-		(pin "4"
-		)
-		(pin "6"
-		)
-		(pin "12"
-		)
-		(pin "5"
-		)
-		(pin "10"
-		)
-		(pin "8"
-		)
-		(pin "7"
-		)
-		(pin "9"
-		)
-		(pin "11"
-		)
-		(instances
-			(project "xr25"
-				(path "/857fcb83-ed52-4e01-bdd2-c0a4a3a1ca9a/646e837e-3db1-4305-b6ca-1f0b46325de9"
-					(reference "U2")
-					(unit 1)
-				)

Commit message: finished first version of pcb
Parts:
- C10, C11: footprint (none) -> Capacitor_SMD:C_1210_3225Metric; LCSC Part # (none) -> C84494
- C4: renamed from C7; footprint (none) -> Capacitor_SMD:C_1206_3216Metric; LCSC Part # (none) -> C51205
- C5: renamed from C6; footprint (none) -> Capacitor_SMD:C_0603_1608Metric; LCSC Part # (none) -> C1622
- C6: renamed from C5; footprint (none) -> Capacitor_SMD:C_0603_1608Metric; LCSC Part # (none) -> C1622
- C7: renamed from C8; footprint (none) -> Capacitor_SMD:C_0603_1608Metric; LCSC Part # (none) -> C15849
- C8: renamed from C4; footprint (none) -> Capacitor_SMD:C_0603_1608Metric; LCSC Part # (none) -> C14663
- C9: footprint (none) -> Capacitor_SMD:C_0603_1608Metric; LCSC Part # (none) -> C61817
- D1: footprint (none) -> lcsc_footprints:C2286_LED-SMD_L1_6-W0_8-R-RD; LCSC Part # (none) -> C2286
- L1: footprint (none) -> lcsc_footprints:C83374_IND-SMD_L6_0-W6_0_SWPA6045S; LCSC Part # (none) -> C83374
- R5: renamed from R3; footprint (none) -> Resistor_SMD:R_0603_1608Metric; LCSC Part # (none) -> C25803
- R6: renamed from R4; footprint (none) -> Resistor_SMD:R_0603_1608Metric; LCSC Part # (none) -> C23053
- R7: renamed from R5; footprint (none) -> Resistor_SMD:R_0603_1608Metric; LCSC Part # (none) -> C4190
- U2: LCSC Part # (none) -> C2863325
