File: hardware/xr25/can_transciever.kicad_sch (KiCad schematic)
At the start: 7 parts, among them J2 Conn_02x02_Odd_Even, U3 PTCAN3404DDFRQ1

Commit message: fixed more ERC issues
Parts:
- CR1: footprint SOT-23_DBZ_TEX -> ESD2CAN24-Q1:SOT-23_DBZ_TEX
- U3: footprint DDF0008A-IPC_A -> TCAN3404-Q1:DDF0008A-IPC_A

Commit message: finished first version of pcb
Parts:
- C14: footprint (none) -> Capacitor_SMD:C_0603_1608Metric; LCSC Part # (none) -> C14663
- CR1: value PESD2CAN24DBZRQ1 -> ESD2CAN24DBZRQ1; LCSC Part # (none) -> C5736151
- D4: footprint (none) -> lcsc_footprints:C125098_LED0603-RD; LCSC Part # (none) -> C125098
- J3: renamed from J2; value Conn_02x02_Odd_Even -> CAN_CONNECTOR; footprint (none) -> lcsc_footprints:C505218_CONN-SMD_430450406
- R8: renamed from R6; footprint (none) -> Resistor_SMD:R_0603_1608Metric; LCSC Part # (none) -> C25804
- R9: renamed from R7; footprint (none) -> Resistor_SMD:R_0603_1608Metric; LCSC Part # (none) -> C4190
- U3: value PTCAN3404DDFRQ1 -> TCAN3404DDFRQ1; LCSC Part # (none) -> C32428067
Changed lines of the file:
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@@
 		(in_pos_files yes)
 		(dnp no)
-		(property "Reference" "#PWR012"
+		(property "Reference" "#PWR015"
 			(at 114.3 76.2 0)
 			(hide yes)
@@
 			(project "xr25"
 				(path "/857fcb83-ed52-4e01-bdd2-c0a4a3a1ca9a/51a7677b-fe14-4c7b-8a2c-af81d60c51a0"
-					(reference "#PWR012")
+					(reference "#PWR015")
 					(unit 1)
 				)
@@
 		(in_pos_files yes)
 		(dnp no)
-		(property "Reference" "R7"
+		(property "Reference" "R9"
 			(at 109.474 123.19 0)
 			(show_name no)
@@
 			)
 		)
-		(property "Footprint" ""
+		(property "Footprint" "Resistor_SMD:R_0603_1608Metric"
 			(at 107.95 124.46 0)
 			(hide yes)
@@
 			)
 		)
+		(property "LCSC Part #" "C4190"
+			(at 107.95 124.46 0)
+			(hide yes)
+			(show_name no)
+			(do_not_autoplace no)
+			(effects
+				(font
+					(size 1.27 1.27)
+				)
+			)
+		)
 		(pin "1"
 		)
@@
 			(project "xr25"
 				(path "/857fcb83-ed52-4e01-bdd2-c0a4a3a1ca9a/51a7677b-fe14-4c7b-8a2c-af81d60c51a0"
-					(reference "R7")
+					(reference "R9")
 					(unit 1)
 				)
@@
 		(dnp no)
 		(fields_autoplaced yes)
-		(property "Reference" "J2"
+		(property "Reference" "J3"
 			(at 210.82 93.98 0)
 			(show_name no)
@@
 			)
 		)
-		(property "Value" "Conn_02x02_Odd_Even"
+		(property "Value" "CAN_CONNECTOR"
 			(at 210.82 96.52 0)
 			(show_name no)
@@
 			)
 		)
-		(property "Footprint" ""
+		(property "Footprint" "lcsc_footprints:C505218_CONN-SMD_430450406"
 			(at 209.55 100.33 0)
 			(hide yes)
@@
 			(project "xr25"
 				(path "/857fcb83-ed52-4e01-bdd2-c0a4a3a1ca9a/51a7677b-fe14-4c7b-8a2c-af81d60c51a0"
-					(reference "J2")
+					(reference "J3")
 					(unit 1)
 				)
@@
 		(dnp no)
 		(fields_autoplaced yes)
-		(property "Reference" "#PWR017"
+		(property "Reference" "#PWR018"
 			(at 217.17 109.22 0)
 			(hide yes)
@@
 			(project "xr25"
 				(path "/857fcb83-ed52-4e01-bdd2-c0a4a3a1ca9a/51a7677b-fe14-4c7b-8a2c-af81d60c51a0"
-					(reference "#PWR017")
+					(reference "#PWR018")
 					(unit 1)
 				)
@@
 		(dnp no)
 		(fields_autoplaced yes)
-		(property "Reference" "#PWR015"
+		(property "Reference" "#PWR016"
 			(at 158.75 121.92 0)
 			(hide yes)
@@
 			(project "xr25"
 				(path "/857fcb83-ed52-4e01-bdd2-c0a4a3a1ca9a/51a7677b-fe14-4c7b-8a2c-af81d60c51a0"
-					(reference "#PWR015")
+					(reference "#PWR016")
 					(unit 1)
 				)
@@
 			)
 		)
-		(property "Value" "PTCAN3404DDFRQ1"
+		(property "Value" "TCAN3404DDFRQ1"
 			(at 140.97 85.09 0)
 			(show_name no)
@@
 		)
 		(property "Description" ""
+			(at 123.19 92.71 0)
+			(hide yes)
+			(show_name no)
+			(do_not_autoplace no)
+			(effects
+				(font
+					(size 1.27 1.27)
+				)
+			)
+		)
+		(property "LCSC Part #" "C32428067"
 			(at 123.19 92.71 0)
 			(hide yes)
@@
 			)
 		)
-		(property "Footprint" ""
+		(property "Footprint" "lcsc_footprints:C125098_LED0603-RD"
 			(at 107.95 118.11 0)
 			(hide yes)
@@
 		(property "Sim.Pins" "1=K 2=A"
 			(at 107.95 118.11 0)
+			(hide yes)
+			(show_name no)
+			(do_not_autoplace no)
+			(effects
+				(font
+					(size 1.27 1.27)
+				)
+			)
+		)
+		(property "LCSC Part #" "C125098"
+			(at 107.95 118.11 90)
 			(hide yes)
 			(show_name no)
@@
 		(dnp no)
 		(fields_autoplaced yes)
-		(property "Reference" "#PWR016"
+		(property "Reference" "#PWR017"
 			(at 194.31 106.68 0)
 			(hide yes)
@@
 			(project "xr25"
 				(path "/857fcb83-ed52-4e01-bdd2-c0a4a3a1ca9a/51a7677b-fe14-4c7b-8a2c-af81d60c51a0"
-					(reference "#PWR016")
+					(reference "#PWR017")
 					(unit 1)
 				)
@@
 		(in_pos_files yes)
 		(dnp no)
-		(property "Reference" "R6"
+		(property "Reference" "R8"
 			(at 109.474 99.06 0)
 			(show_name no)
@@
 			)
 		)
-		(property "Footprint" ""
+		(property "Footprint" "Resistor_SMD:R_0603_1608Metric"
 			(at 107.95 100.33 0)
 			(hide yes)
@@
 			)
 		)
+		(property "LCSC Part #" "C25804"
+			(at 107.95 100.33 0)
+			(hide yes)
+			(show_name no)
+			(do_not_autoplace no)
+			(effects
+				(font
+					(size 1.27 1.27)
+				)
+			)
+		)
 		(pin "1"
 		)
@@
 			(project "xr25"
 				(path "/857fcb83-ed52-4e01-bdd2-c0a4a3a1ca9a/51a7677b-fe14-4c7b-8a2c-af81d60c51a0"
-					(reference "R6")
+					(reference "R8")
 					(unit 1)
 				)
@@
 			)
 		)
-		(property "Footprint" ""
+		(property "Footprint" "Capacitor_SMD:C_0603_1608Metric"
 			(at 114.3 85.09 0)
 			(hide yes)
@@
 			)
 		)
+		(property "LCSC Part #" "C14663"
+			(at 114.3 85.09 0)
+			(hide yes)
+			(show_name no)
+			(do_not_autoplace no)
+			(effects
+				(font
+					(size 1.27 1.27)
+				)
+			)
+		)
 		(pin "2"
 		)
@@
 				(path "/857fcb83-ed52-4e01-bdd2-c0a4a3a1ca9a/51a7677b-fe14-4c7b-8a2c-af81d60c51a0"
 					(reference "C14")
+					(unit 1)
+				)
+			)
+		)
+	)
+	(symbol
+		(lib_id "ESD2CAN24-Q1:PESD2CAN24DBZRQ1")
+		(at 171.45 100.33 0)
+		(unit 1)
+		(body_style 1)
+		(exclude_from_sim no)
+		(in_bom yes)
+		(on_board yes)
+		(in_pos_files yes)
+		(dnp no)
+		(fields_autoplaced yes)
+		(property "Reference" "CR1"
+			(at 182.88 92.71 0)
+			(show_name no)
+			(do_not_autoplace no)
+			(effects
+				(font
+					(size 1.524 1.524)
+				)
+			)
+		)
+		(property "Value" "ESD2CAN24DBZRQ1"
+			(at 182.88 95.25 0)
+			(show_name no)
+			(do_not_autoplace no)
+			(effects
+				(font
+					(size 1.524 1.524)
+				)
+			)
+		)
+		(property "Footprint" "ESD2CAN24-Q1:SOT-23_DBZ_TEX"
+			(at 171.45 100.33 0)
+			(hide yes)
+			(show_name no)
+			(do_not_autoplace no)
+			(effects
+				(font
+					(size 1.27 1.27)
+					(italic yes)
+				)
+			)
+		)
+		(property "Datasheet" "ESD2CAN24DBZRQ1"
+			(at 171.45 100.33 0)
+			(hide yes)
+			(show_name no)
+			(do_not_autoplace no)
+			(effects
+				(font
+					(size 1.27 1.27)
+					(italic yes)
+				)
+			)
+		)
+		(property "Description" ""
+			(at 171.45 100.33 0)
+			(hide yes)
+			(show_name no)
+			(do_not_autoplace no)
+			(effects
+				(font
+					(size 1.27 1.27)
+				)
+			)
+		)
+		(property "LCSC Part #" "C5736151"
+			(at 171.45 100.33 0)
+			(hide yes)
+			(show_name no)
+			(do_not_autoplace no)
+			(effects
+				(font
+					(size 1.27 1.27)
+				)
+			)
+		)
+		(pin "1"
+		)
+		(pin "2"
+		)
+		(pin "3"
+		)
+		(instances
+			(project "xr25"
+				(path "/857fcb83-ed52-4e01-bdd2-c0a4a3a1ca9a/51a7677b-fe14-4c7b-8a2c-af81d60c51a0"
+					(reference "CR1")
 					(unit 1)
 				)
@@
 		(dnp no)
 		(fields_autoplaced yes)
-		(property "Reference" "#PWR013"
+		(property "Reference" "#PWR014"
 			(at 107.95 109.22 0)
 			(hide yes)
@@
 			(project "xr25"
 				(path "/857fcb83-ed52-4e01-bdd2-c0a4a3a1ca9a/51a7677b-fe14-4c7b-8a2c-af81d60c51a0"
-					(reference "#PWR013")
-					(unit 1)
-				)
-			)
-		)
-	)
-	(symbol
-		(lib_id "ESD2CAN24-Q1:PESD2CAN24DBZRQ1")
-		(at 171.45 100.33 0)
-		(unit 1)
-		(body_style 1)
-		(exclude_from_sim no)
-		(in_bom yes)
-		(on_board yes)
-		(in_pos_files yes)
-		(dnp no)
-		(fields_autoplaced yes)
-		(property "Reference" "CR1"
-			(at 182.88 92.71 0)
-			(show_name no)
-			(do_not_autoplace no)
-			(effects
-				(font
-					(size 1.524 1.524)
-				)
-			)
-		)
-		(property "Value" "PESD2CAN24DBZRQ1"
-			(at 182.88 95.25 0)
-			(show_name no)
-			(do_not_autoplace no)
-			(effects
-				(font
-					(size 1.524 1.524)
-				)
-			)
-		)
-		(property "Footprint" "ESD2CAN24-Q1:SOT-23_DBZ_TEX"
-			(at 171.45 100.33 0)
-			(hide yes)
-			(show_name no)
-			(do_not_autoplace no)
-			(effects
-				(font
-					(size 1.27 1.27)
-					(italic yes)
-				)
-			)
-		)
-		(property "Datasheet" "PESD2CAN24DBZRQ1"
-			(at 171.45 100.33 0)
-			(hide yes)
-			(show_name no)
-			(do_not_autoplace no)
-			(effects
-				(font
-					(size 1.27 1.27)
-					(italic yes)
-				)
-			)
-		)
-		(property "Description" ""
-			(at 171.45 100.33 0)
-			(hide yes)
-			(show_name no)
-			(do_not_autoplace no)
-			(effects
-				(font
-					(size 1.27 1.27)
-				)
-			)
-		)
-		(pin "2"
-		)
-		(pin "1"
-		)
-		(pin "3"
-		)
-		(instances
-			(project "xr25"
-				(path "/857fcb83-ed52-4e01-bdd2-c0a4a3a1ca9a/51a7677b-fe14-4c7b-8a2c-af81d60c51a0"
-					(reference "CR1")
-					(unit 1)
-				)
+					(reference "#PWR014")
+					(unit 1)
+				)
