File: hardware/xr25/esp32.kicad_sch (KiCad schematic)
At the start: 12 parts, among them J1 Conn_02x03_Odd_Even, U1 ESP32-C3-WROOM-02

Commit message: fixed more ERC issues
Changed lines of the file:
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@@
 	(wire
 		(pts
-			(xy 152.4 49.53) (xy 107.95 49.53)
+			(xy 107.95 49.53) (xy 152.4 49.53)
 		)
 		(stroke

Commit message: finished first version of pcb
Parts:
- removed TP2: GND, symbol Connector:TestPoint
- added R2, R3: 10k, Resistor_SMD:R_0603_1608Metric, symbol Device:R_Small
- C1: renamed from C3; footprint (none) -> Capacitor_SMD:C_0603_1608Metric; LCSC Part # (none) -> C15849
- C2: footprint (none) -> Capacitor_SMD:C_0603_1608Metric; LCSC Part # (none) -> C14663
- C3: renamed from C1; footprint (none) -> Capacitor_SMD:C_0805_2012Metric; LCSC Part # (none) -> C15850
- J2: renamed from J1; value Conn_02x03_Odd_Even -> PROGRAMMER_HEADER; footprint (none) -> Connector_PinHeader_2.54mm:PinHeader_2x03_P2.54mm_Vertical; now not fitted
- R1: renamed from R2; footprint (none) -> Resistor_SMD:R_0603_1608Metric; LCSC Part # (none) -> C25804
- R4: renamed from R1; footprint (none) -> Resistor_SMD:R_0603_1608Metric; LCSC Part # (none) -> C25804
- TP1: renamed from TP5; footprint (none) -> TestPoint:TestPoint_Pad_D1.5mm
- TP2: renamed from TP4; footprint (none) -> TestPoint:TestPoint_Pad_D1.5mm
- TP3: renamed from TP1; footprint (none) -> TestPoint:TestPoint_Pad_D1.5mm
- TP4: renamed from TP3; footprint (none) -> TestPoint:TestPoint_Pad_D1.5mm
- U1: LCSC Part # (none) -> C2934560
Connections:
- net 3V3_RAIL: now also R2.1, R3.1
- net at U1.16 (IO2): now also R3.2
- net at U1.7 (IO8): now also R2.2
- no-connect marks 8 -> 6
Other:
- moved on the sheet: C1, C2, C3, R1, R4, TP1, TP2, TP3, TP4, U1
