File: hardware/xr25/protection_circuit.kicad_sch (KiCad schematic)
At the start: 5 parts

Commit message: fixed more ERC issues
Changed lines of the file:
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@@
+	)
+	(junction
+		(at 175.26 96.52)
+		(diameter 0)
+		(color 0 0 0 0)
 	)
 	(junction
@@
 	(wire
 		(pts
+			(xy 175.26 96.52) (xy 176.53 96.52)
+		)
+		(stroke
+			(width 0)
+			(type default)
+		)
+	)
+	(wire
+		(pts
 			(xy 153.67 90.17) (xy 153.67 87.63)
 		)
@@
 	(wire
 		(pts
-			(xy 163.83 96.52) (xy 176.53 96.52)
+			(xy 163.83 96.52) (xy 175.26 96.52)
 		)
 		(stroke
@@
 					(unit 1)
 				)
+			)
+		)
+	)
+	(symbol
+		(lib_id "power:PWR_FLAG")
+		(at 175.26 96.52 0)
+		(unit 1)
+		(body_style 1)
+		(exclude_from_sim no)
+		(in_bom yes)
+		(on_board yes)
+		(in_pos_files yes)
+		(dnp no)
+		(fields_autoplaced yes)
+		(property "Reference" "#FLG02"
+			(at 175.26 94.615 0)
+			(hide yes)
+			(show_name no)
+			(do_not_autoplace no)
+			(effects
+				(font
+					(size 1.27 1.27)
+				)
+			)
+		)
+		(property "Value" "PWR_FLAG"
+			(at 175.26 91.44 0)
+			(hide yes)
+			(show_name no)
+			(do_not_autoplace no)
+			(effects
+				(font
+					(size 1.27 1.27)
+				)
+			)
+		)
+		(property "Footprint" ""
+			(at 175.26 96.52 0)
+			(hide yes)
+			(show_name no)
+			(do_not_autoplace no)
+			(effects
+				(font
+					(size 1.27 1.27)
+				)
+			)
+		)
+		(property "Datasheet" ""
+			(at 175.26 96.52 0)
+			(hide yes)
+			(show_name no)
+			(do_not_autoplace no)
+			(effects
+				(font
+					(size 1.27 1.27)
+				)
+			)
+		)
+		(property "Description" "Special symbol for telling ERC where power comes from"
+			(at 175.26 96.52 0)
+			(hide yes)
+			(show_name no)
+			(do_not_autoplace no)
+			(effects
+				(font
+					(size 1.27 1.27)
+				)
+			)
+		)
+		(pin "1"
+		)
+		(instances
+			(project "xr25"
+				(path "/857fcb83-ed52-4e01-bdd2-c0a4a3a1ca9a/11319032-47b5-4b16-a093-272a5d49cb5c"
+					(reference "#FLG02")
+					(unit 1)
+				)

Commit message: finished first version of pcb
Parts:
- C12: footprint (none) -> Capacitor_SMD:C_1210_3225Metric; LCSC Part # (none) -> C49296968
- C13: footprint (none) -> Capacitor_SMD:C_0805_2012Metric; LCSC Part # (none) -> C28233
- D2: footprint Diode_SMD:D_SMB -> lcsc_footprints:C425875_SMB_L4_3-W3_6-LS5_4-BI; LCSC Part # (none) -> C425875
- D3: footprint (none) -> lcsc_footprints:C2969868_SOD-123FL_L2_6-W1_6-LS3_5-FD; LCSC Part # (none) -> C2969868
- TH1: footprint (none) -> lcsc_footprints:C910836_F2018; LCSC Part # (none) -> C910836
Changed lines of the file:
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@@
 		(in_pos_files yes)
 		(dnp no)
-		(property "Reference" "#PWR011"
+		(property "Reference" "#PWR013"
 			(at 158.75 80.01 0)
 			(hide yes)
@@
 			(project "xr25"
 				(path "/857fcb83-ed52-4e01-bdd2-c0a4a3a1ca9a/11319032-47b5-4b16-a093-272a5d49cb5c"
-					(reference "#PWR011")
+					(reference "#PWR013")
 					(unit 1)
 				)
@@
 			)
 		)
-		(property "Footprint" ""
+		(property "Footprint" "lcsc_footprints:C910836_F2018"
 			(at 113.03 97.79 0)
 			(hide yes)
@@
 		(property "Description" "Temperature dependent resistor, positive temperature coefficient"
 			(at 118.11 96.52 0)
+			(hide yes)
+			(show_name no)
+			(do_not_autoplace no)
+			(effects
+				(font
+					(size 1.27 1.27)
+				)
+			)
+		)
+		(property "LCSC Part #" "C910836"
+			(at 118.11 96.52 90)
 			(hide yes)
 			(show_name no)
@@
 			)
 		)
-		(property "Footprint" ""
+		(property "Footprint" "lcsc_footprints:C2969868_SOD-123FL_L2_6-W1_6-LS3_5-FD"
 			(at 142.24 96.52 0)
 			(hide yes)
@@
 		)
 		(property "Description" "Schottky diode"
+			(at 142.24 96.52 0)
+			(hide yes)
+			(show_name no)
+			(do_not_autoplace no)
+			(effects
+				(font
+					(size 1.27 1.27)
+				)
+			)
+		)
+		(property "LCSC Part #" "C2969868"
 			(at 142.24 96.52 0)
 			(hide yes)
@@
 		(dnp no)
 		(fields_autoplaced yes)
-		(property "Reference" "#FLG02"
+		(property "Reference" "#FLG04"
 			(at 175.26 94.615 0)
 			(hide yes)
@@
 			(project "xr25"
 				(path "/857fcb83-ed52-4e01-bdd2-c0a4a3a1ca9a/11319032-47b5-4b16-a093-272a5d49cb5c"
-					(reference "#FLG02")
+					(reference "#FLG04")
 					(unit 1)
 				)
@@
 			)
 		)
-		(property "Footprint" "Diode_SMD:D_SMB"
+		(property "Footprint" "lcsc_footprints:C425875_SMB_L4_3-W3_6-LS5_4-BI"
 			(at 134.62 100.33 0)
 			(hide yes)
@@
 		(property "Description" "600W bidirectional Transient Voltage Suppressor, 33.0Vr, SMA(DO-214AC)"
 			(at 129.54 100.33 0)
+			(hide yes)
+			(show_name no)
+			(do_not_autoplace no)
+			(effects
+				(font
+					(size 1.27 1.27)
+				)
+			)
+		)
+		(property "LCSC Part #" "C425875"
+			(at 129.54 100.33 90)
 			(hide yes)
 			(show_name no)
@@
 			)
 		)
-		(property "Footprint" ""
+		(property "Footprint" "Capacitor_SMD:C_1210_3225Metric"
 			(at 153.67 92.71 0)
 			(hide yes)
@@
 		)
 		(property "Description" "Unpolarized capacitor, small symbol"
+			(at 153.67 92.71 0)
+			(hide yes)
+			(show_name no)
+			(do_not_autoplace no)
+			(effects
+				(font
+					(size 1.27 1.27)
+				)
+			)
+		)
+		(property "LCSC Part #" "C49296968"
 			(at 153.67 92.71 0)
 			(hide yes)
@@
 			)
 		)
-		(property "Footprint" ""
+		(property "Footprint" "Capacitor_SMD:C_0805_2012Metric"
 			(at 163.83 92.71 0)
 			(hide yes)
@@
 		)
 		(property "Description" "Unpolarized capacitor, small symbol"
+			(at 163.83 92.71 0)
+			(hide yes)
+			(show_name no)
+			(do_not_autoplace no)
+			(effects
+				(font
+					(size 1.27 1.27)
+				)
+			)
+		)
+		(property "LCSC Part #" "C28233"
 			(at 163.83 92.71 0)
 			(hide yes)
@@
 		(dnp no)
 		(fields_autoplaced yes)
-		(property "Reference" "#PWR010"
+		(property "Reference" "#PWR012"
 			(at 129.54 111.76 0)
 			(hide yes)
@@
 			(project "xr25"
 				(path "/857fcb83-ed52-4e01-bdd2-c0a4a3a1ca9a/11319032-47b5-4b16-a093-272a5d49cb5c"
-					(reference "#PWR010")
-					(unit 1)
-				)
+					(reference "#PWR012")
+					(unit 1)
+				)
