File: hardware/xr25/xr25.kicad_sch (KiCad schematic)
At the start: 1 part, among them J3 XR25_INTERFACE

Commit message: expanded main pcb schematics
Other:
- sheet CAN Transciever: file can_transcieverkicad_sch.kicad_sch -> can_transciever.kicad_sch
Changed lines of the file:
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@@
 			)
 		)
-		(property "Sheetfile" "can_transcieverkicad_sch.kicad_sch"
+		(property "Sheetfile" "can_transciever.kicad_sch"
 			(at 177.8 116.1546 0)
 			(show_name no)

Commit message: fixed more ERC issues
Changed lines of the file:
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@@
 		(color 0 0 0 0)
 	)
+	(junction
+		(at 130.81 66.04)
+		(diameter 0)
+		(color 0 0 0 0)
+	)
 	(wire
 		(pts
@@
 	(wire
 		(pts
+			(xy 146.05 57.15) (xy 177.8 57.15)
+		)
+		(stroke
+			(width 0)
+			(type default)
+		)
+	)
+	(wire
+		(pts
 			(xy 60.96 85.09) (xy 68.58 85.09)
 		)
@@
 	(wire
 		(pts
-			(xy 146.05 57.15) (xy 177.8 57.15)
-		)
-		(stroke
-			(width 0)
-			(type default)
-		)
-	)
-	(wire
-		(pts
 			(xy 153.67 109.22) (xy 153.67 85.09)
 		)
@@
 	(wire
 		(pts
+			(xy 130.81 66.04) (xy 60.96 66.04)
+		)
+		(stroke
+			(width 0)
+			(type default)
+		)
+	)
+	(wire
+		(pts
 			(xy 201.93 87.63) (xy 208.28 87.63)
 		)
@@
 	(wire
 		(pts
-			(xy 140.97 66.04) (xy 60.96 66.04)
+			(xy 140.97 66.04) (xy 130.81 66.04)
 		)
 		(stroke
@@
 					(unit 1)
 				)
+			)
+		)
+	)
+	(symbol
+		(lib_id "power:PWR_FLAG")
+		(at 130.81 66.04 0)
+		(unit 1)
+		(body_style 1)
+		(exclude_from_sim no)
+		(in_bom yes)
+		(on_board yes)
+		(in_pos_files yes)
+		(dnp no)
+		(fields_autoplaced yes)
+		(property "Reference" "#FLG01"
+			(at 130.81 64.135 0)
+			(hide yes)
+			(show_name no)
+			(do_not_autoplace no)
+			(effects
+				(font
+					(size 1.27 1.27)
+				)
+			)
+		)
+		(property "Value" "PWR_FLAG"
+			(at 130.81 60.96 0)
+			(hide yes)
+			(show_name no)
+			(do_not_autoplace no)
+			(effects
+				(font
+					(size 1.27 1.27)
+				)
+			)
+		)
+		(property "Footprint" ""
+			(at 130.81 66.04 0)
+			(hide yes)
+			(show_name no)
+			(do_not_autoplace no)
+			(effects
+				(font
+					(size 1.27 1.27)
+				)
+			)
+		)
+		(property "Datasheet" ""
+			(at 130.81 66.04 0)
+			(hide yes)
+			(show_name no)
+			(do_not_autoplace no)
+			(effects
+				(font
+					(size 1.27 1.27)
+				)
+			)
+		)
+		(property "Description" "Special symbol for telling ERC where power comes from"
+			(at 130.81 66.04 0)
+			(hide yes)
+			(show_name no)
+			(do_not_autoplace no)
+			(effects
+				(font
+					(size 1.27 1.27)
+				)
+			)
+		)
+		(pin "1"
+		)
+		(instances
+			(project "xr25"
+				(path "/857fcb83-ed52-4e01-bdd2-c0a4a3a1ca9a"
+					(reference "#FLG01")
+					(unit 1)
+				)

Commit message: finished first version of pcb
Parts:
- J1: renamed from J3; footprint (none) -> Connector_PinHeader_2.54mm:PinHeader_2x03_P2.54mm_Vertical; symbol Connector:Conn_01x03_Pin -> Connector_Generic:Conn_02x03_Odd_Even; now not fitted
Connections:
- net GND: now also J1.3 (Pin_3), J1.4 (Pin_4); no longer J1.2 (Pin_2)
- net Protection Circuit/VBAT: now also J1.2 (Pin_2); no longer J1.1 (Pin_1)
- net XR25 Input/XR25_INPUT: now also J1.6 (Pin_6); no longer J1.3 (Pin_3)
- no-connect marks 0 -> 2

Commit message: finished rev 1.1 of plug pcb
Connections:
- net Protection Circuit/VBAT: now also J1.1 (Pin_1)
- no-connect marks 2 -> 1
Changed lines of the file:
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@@
+	)
+	(junction
+		(at 140.97 59.69)
+		(diameter 0)
+		(color 0 0 0 0)
 	)
 	(junction
@@
 	)
 	(no_connect
-		(at 140.97 41.91)
-	)
-	(no_connect
 		(at 146.05 41.91)
 	)
@@
 	(wire
 		(pts
+			(xy 140.97 59.69) (xy 140.97 66.04)
+		)
+		(stroke
+			(width 0)
+			(type default)
+		)
+	)
+	(wire
+		(pts
 			(xy 144.78 85.09) (xy 153.67 85.09)
 		)
@@
 	(wire
 		(pts
+			(xy 137.16 59.69) (xy 140.97 59.69)
+		)
+		(stroke
+			(width 0)
+			(type default)
+		)
+	)
+	(wire
+		(pts
 			(xy 60.96 85.09) (xy 68.58 85.09)
 		)
@@
 	(wire
 		(pts
-			(xy 140.97 54.61) (xy 140.97 66.04)
+			(xy 140.97 54.61) (xy 140.97 59.69)
+		)
+		(stroke
+			(width 0)
+			(type default)
+		)
+	)
+	(wire
+		(pts
+			(xy 137.16 41.91) (xy 137.16 59.69)
 		)
 		(stroke
@@
 		)
 		(stroke
+			(width 0)
+			(type default)
+		)
+	)
+	(wire
+		(pts
+			(xy 140.97 41.91) (xy 137.16 41.91)
+		)
+		(stroke
